File: cc2652r.brd (EAGLE design)
At the start: 25.3 x 43.9 mm, 38 parts, among them IC2 CP2102, J3 CORTEX_DEBUG_SMD, J5 TYPE-C-31-M-12, Q2 SI2323DS, U1 RF-BM-2652B1, U2 3.3V

Commit message: Add files via upload
Parts:
- moved R11 2.02 mm to (18.7, 14.4), turned to 270 degrees
- moved C4 0.76 mm to (17.3, 15.1)
- moved R8 0.70 mm to (15.9, 15.7)
- moved D4 0.23 mm to (20.3, 14.9), turned to 270 degrees
Connections:
- net RST: now also J2.1
- net U3V3: no longer J2.1
Routing:
- net U3V3: track 21.4 -> 7.14 mm
- net RST: track 75.6 -> 81.4 mm
- net N$8: track 1.54 -> 2.28 mm
- net N$1: track 2.49 -> 1.79 mm
- net +5V: track 37.8 -> 37.1 mm
Other:
- board text added: "RST"
