File: cc2652r.sch (EAGLE design)
At the start: 38 parts, among them IC2 CP2102, J3 CORTEX_DEBUG_SMD, J5 TYPE-C-31-M-12, Q2 SI2323DS, U1 RF-BM-2652B1, U2 3.3V

Commit message: Add files via upload
Connections:
- net RST: now also J2.1
- net U3V3: no longer J2.1
Changed lines of the file:
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@@
 <pinref part="C4" gate="G$1" pin="1"/>
 <wire x1="60.96" y1="35.56" x2="60.96" y2="33.02" width="0.1524" layer="91"/>
-<pinref part="IC2" gate="G$1" pin="VDD"/>
 <wire x1="60.96" y1="33.02" x2="68.58" y2="33.02" width="0.1524" layer="91"/>
 <pinref part="R11" gate="G$1" pin="2"/>
+<pinref part="IC2" gate="G$1" pin="VDD"/>
 <wire x1="68.58" y1="33.02" x2="83.82" y2="33.02" width="0.1524" layer="91"/>
 <junction x="68.58" y="33.02"/>
-<label x="78.74" y="33.02" size="1.778" layer="95"/>
-</segment>
-<segment>
-<pinref part="J2" gate="G$1" pin="1"/>
-<wire x1="294.64" y1="38.1" x2="299.72" y2="38.1" width="0.1524" layer="91"/>
-<label x="294.64" y="38.1" size="1.778" layer="95"/>
 </segment>
 </net>
@@
 <label x="177.8" y="22.86" size="1.778" layer="95"/>
 </segment>
+<segment>
+<pinref part="J2" gate="G$1" pin="1"/>
+<wire x1="294.64" y1="38.1" x2="299.72" y2="38.1" width="0.1524" layer="91"/>
+<label x="294.64" y="38.1" size="1.778" layer="95"/>
+</segment>
 </net>
